Commit message: changes spheroid to have 8 rotors to cover all DOF and added yaml

File: marinegym/robots/assets/urdf/Spheroid/Spheroid.urdf (robot description, URDF)
Before this commit: robot Spheroid, 5 links, 4 joints
Links:
- added link rotor_4, mass 0.01; visual cylinder length=0.02 radius=0.04
- added link rotor_5, mass 0.01; visual cylinder length=0.02 radius=0.04
- added link rotor_6, mass 0.01; visual cylinder length=0.02 radius=0.04
- added link rotor_7, mass 0.01; visual cylinder length=0.02 radius=0.04
- link base_link: mass 129.9740 -> 130.2940
- link rotor_0: mass 0.1 -> 0.01; geometry visual cylinder length=0.02 radius=0.04
- link rotor_1: mass 0.1 -> 0.01; geometry visual cylinder length=0.02 radius=0.04
- link rotor_2: mass 0.1 -> 0.01; geometry visual cylinder length=0.02 radius=0.04
- link rotor_3: mass 0.1 -> 0.01; geometry visual cylinder length=0.02 radius=0.04
Joints:
- added joint rotor_4_joint: type continuous, parent base_link, child rotor_4, origin xyz=0.250000 0.216506 0.000000 rpy=-0.000000 -0.000000 -0.785398, axis 1 0 0
- added joint rotor_5_joint: type continuous, parent base_link, child rotor_5, origin xyz=0.250000 -0.216506 0.000000 rpy=0.000000 -0.000000 0.785398, axis 1 0 0
- added joint rotor_6_joint: type continuous, parent base_link, child rotor_6, origin xyz=-0.250000 -0.216506 0.000000 rpy=-0.000000 -0.000000 -0.785398, axis 1 0 0
- added joint rotor_7_joint: type continuous, parent base_link, child rotor_7, origin xyz=-0.250000 0.216506 0.000000 rpy=0.000000 -0.000000 0.785398, axis 1 0 0
- joint rotor_0_joint: axis 0 0 1 -> 1 0 0; origin xyz=0.400000 0.150000 0.000000 rpy=0 0 0 -> xyz=0.400000 0.150000 0.000000 rpy=0.000000 -1.570796 -3.141593
- joint rotor_1_joint: axis 0 0 1 -> 1 0 0; origin xyz=0.400000 -0.150000 0.000000 rpy=0 0 0 -> xyz=0.400000 -0.150000 0.000000 rpy=0.000000 -1.570796 -3.141593
- joint rotor_2_joint: axis 0 0 1 -> 1 0 0; origin xyz=-0.400000 -0.150000 0.000000 rpy=0 0 0 -> xyz=-0.400000 -0.150000 0.000000 rpy=0.000000 -1.570796 -3.141593
- joint rotor_3_joint: axis 0 0 1 -> 1 0 0; origin xyz=-0.400000 0.150000 0.000000 rpy=0 0 0 -> xyz=-0.400000 0.150000 0.000000 rpy=0.000000 -1.570796 -3.141593
